Commit message: 加入python3.9支持的真实机械臂控制代码，加入本地回环通信接受start信息，修改urdf文件，加入侧视图urdf文件，修改gripper配置文件，修改服务器代码，加入键盘控制代码，修改工具函数，加入仿真环境控制代码，修改python3.8和python3.9的控制代码

File: ace_teleop/assets/gen_72_b_description/urdf/GEN72_franka_side.urdf (robot description, URDF)
Before this commit: robot GEN72, 29 links, 28 joints
Links:
- link l_panda_hand: geometry collision mesh filename=../../franka/franka_description/meshes/collision/hand.stl; visual mesh filename=../../franka/franka_description/meshes/visual/hand.glb
- link l_panda_leftfinger: geometry collision mesh filename=../../franka/franka_description/meshes/collision/finger.stl; visual mesh filename=../../franka/franka_description/meshes/visual/finger.glb
- link l_panda_rightfinger: geometry collision mesh filename=../../franka/franka_description/meshes/collision/finger.stl; visual mesh filename=../../franka/franka_description/meshes/visual/finger.glb
- link r_panda_hand: geometry collision mesh filename=../../franka/franka_description/meshes/collision/hand.stl; visual mesh filename=../../franka/franka_description/meshes/visual/hand.glb
- link r_panda_leftfinger: geometry collision mesh filename=../../franka/franka_description/meshes/collision/finger.stl; visual mesh filename=../../franka/franka_description/meshes/visual/finger.glb
- link r_panda_rightfinger: geometry collision mesh filename=../../franka/franka_description/meshes/collision/finger.stl; visual mesh filename=../../franka/franka_description/meshes/visual/finger.glb
Joints:
- joint l_base_joint: origin xyz=0 0.35 0 rpy=0 0 0 -> xyz=0 0.1 0 rpy=-1.5708 0 0
- joint r_base_joint: origin xyz=0 -0.35 0 rpy=0 0 0 -> xyz=0 -0.1 0 rpy=1.5708 0 0
