Commit message: 更新代码,删除了不必要的信息

File: ace_teleop/assets/gen_72_b_description/urdf/GEN72_franka.urdf (robot description, URDF)
Before this commit: robot GEN72, 29 links, 28 joints
Links:
- link l_Link1: geometry collision mesh filename=/home/s402/ACE/ACETeleop-main/ace_teleop/assets/gen_72_b_de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; visual mesh filename=/home/s402/ACE/ACETeleop-main/ace_teleop/assets/gen_72_b_de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
- link l_Link2: geometry collision mesh filename=/home/s402/ACE/ACETeleop-main/ace_teleop/assets/gen_72_b_de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; visual mesh filename=/home/s402/ACE/ACETeleop-main/ace_teleop/assets/gen_72_b_de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
- link l_Link3: geometry collision mesh filename=/home/s402/ACE/ACETeleop-main/ace_teleop/assets/gen_72_b_de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; visual mesh filename=/home/s402/ACE/ACETeleop-main/ace_teleop/assets/gen_72_b_de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
- link l_Link4: geometry collision mesh filename=/home/s402/ACE/ACETeleop-main/ace_teleop/assets/gen_72_b_de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; visual mesh filename=/home/s402/ACE/ACETeleop-main/ace_teleop/assets/gen_72_b_de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
- link l_Link5: geometry collision mesh filename=/home/s402/ACE/ACETeleop-main/ace_teleop/assets/gen_72_b_de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; visual mesh filename=/home/s402/ACE/ACETeleop-main/ace_teleop/assets/gen_72_b_de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
- link l_Link6: geometry collision mesh filename=/home/s402/ACE/ACETeleop-main/ace_teleop/assets/gen_72_b_de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; visual mesh filename=/home/s402/ACE/ACETeleop-main/ace_teleop/assets/gen_72_b_de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
- link l_Link7: geometry collision mesh filename=/home/s402/ACE/ACETeleop-main/ace_teleop/assets/gen_72_b_de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; visual mesh filename=/home/s402/ACE/ACETeleop-main/ace_teleop/assets/gen_72_b_de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
- link l_base_link: geometry collision mesh filename=/home/s402/ACE/ACETeleop-main/ace_teleop/assets/gen_72_b_de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; visual mesh filename=/home/s402/ACE/ACETeleop-main/ace_teleop/assets/gen_72_b_de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
- link l_panda_hand: geometry collision mesh filename=/home/s402/ACE/ACETeleop-main/ace_teleop/assets/franka/fran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; visual mesh filename=/home/s402/ACE/ACETeleop-main/ace_teleop/assets/franka/fran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
- link r_Link1: geometry collision mesh filename=/home/s402/ACE/ACETeleop-main/ace_teleop/assets/gen_72_b_de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; visual mesh filename=/home/s402/ACE/ACETeleop-main/ace_teleop/assets/gen_72_b_de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
- link r_Link2: geometry collision mesh filename=/home/s402/ACE/ACETeleop-main/ace_teleop/assets/gen_72_b_de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; visual mesh filename=/home/s402/ACE/ACETeleop-main/ace_teleop/assets/gen_72_b_de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
- link r_Link3: geometry collision mesh filename=/home/s402/ACE/ACETeleop-main/ace_teleop/assets/gen_72_b_de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; visual mesh filename=/home/s402/ACE/ACETeleop-main/ace_teleop/assets/gen_72_b_de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
- link r_Link4: geometry collision mesh filename=/home/s402/ACE/ACETeleop-main/ace_teleop/assets/gen_72_b_de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; visual mesh filename=/home/s402/ACE/ACETeleop-main/ace_teleop/assets/gen_72_b_de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
- link r_Link5: geometry collision mesh filename=/home/s402/ACE/ACETeleop-main/ace_teleop/assets/gen_72_b_de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; visual mesh filename=/home/s402/ACE/ACETeleop-main/ace_teleop/assets/gen_72_b_de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
- link r_Link6: geometry collision mesh filename=/home/s402/ACE/ACETeleop-main/ace_teleop/assets/gen_72_b_de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; visual mesh filename=/home/s402/ACE/ACETeleop-main/ace_teleop/assets/gen_72_b_de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
- link r_Link7: geometry collision mesh filename=/home/s402/ACE/ACETeleop-main/ace_teleop/assets/gen_72_b_de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; visual mesh filename=/home/s402/ACE/ACETeleop-main/ace_teleop/assets/gen_72_b_de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
- link r_base_link: geometry collision mesh filename=/home/s402/ACE/ACETeleop-main/ace_teleop/assets/gen_72_b_de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; visual mesh filename=/home/s402/ACE/ACETeleop-main/ace_teleop/assets/gen_72_b_de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
